File: pcb/kicad/ic_5v_to_3v3.kicad_sch (KiCad schematic)
At the start: 3 parts, among them U2 AMS1117-3.3

Commit message: rev3-update
Parts:
- U2: footprint Package_TO_SOT_SMD:TO-252-2 -> Package_TO_SOT_SMD:SOT-223-3_TabPin2
Changed lines of the file:
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@@
   (title_block
     (title "Kwartzlab Environmental Sensor")
-    (date "2023-04-04")
-    (rev "2")
+    (date "2023-04-20")
+    (rev "3")
     (company "Created By: Erin Reed (FireLabs - www.firelabs.ca)")
   )
@@
     (pin "1")
     (instances
-      (project "KwartzLab-SensorBoard-Rev2"
+      (project "KwartzLab-SensorBoard-Rev3"
         (path "/02789d54-6086-45b9-8196-8325e6f33099/6c6a6a4b-14a8-444c-aff8-64b652436e04"
           (reference "#PWR018") (unit 1)
@@
     (pin "2")
     (instances
-      (project "KwartzLab-SensorBoard-Rev2"
+      (project "KwartzLab-SensorBoard-Rev3"
         (path "/02789d54-6086-45b9-8196-8325e6f33099/6c6a6a4b-14a8-444c-aff8-64b652436e04"
           (reference "C5") (unit 1)
@@
     (pin "1")
     (instances
-      (project "KwartzLab-SensorBoard-Rev2"
+      (project "KwartzLab-SensorBoard-Rev3"
         (path "/02789d54-6086-45b9-8196-8325e6f33099/6c6a6a4b-14a8-444c-aff8-64b652436e04"
           (reference "#PWR020") (unit 1)
@@
     (pin "2")
     (instances
-      (project "KwartzLab-SensorBoard-Rev2"
+      (project "KwartzLab-SensorBoard-Rev3"
         (path "/02789d54-6086-45b9-8196-8325e6f33099/6c6a6a4b-14a8-444c-aff8-64b652436e04"
           (reference "C4") (unit 1)
@@
     (pin "1")
     (instances
-      (project "KwartzLab-SensorBoard-Rev2"
+      (project "KwartzLab-SensorBoard-Rev3"
         (path "/02789d54-6086-45b9-8196-8325e6f33099/6c6a6a4b-14a8-444c-aff8-64b652436e04"
           (reference "#PWR019") (unit 1)
@@
       (effects (font (size 1.27 1.27)))
     )
-    (property "Footprint" "Package_TO_SOT_SMD:TO-252-2" (at 143.51 83.82 0)
+    (property "Footprint" "Package_TO_SOT_SMD:SOT-223-3_TabPin2" (at 143.51 83.82 0)
       (effects (font (size 1.27 1.27)) hide)
     )
@@
     (pin "3")
     (instances
-      (project "KwartzLab-SensorBoard-Rev2"
+      (project "KwartzLab-SensorBoard-Rev3"
         (path "/02789d54-6086-45b9-8196-8325e6f33099/6c6a6a4b-14a8-444c-aff8-64b652436e04"
           (reference "U2") (unit 1)
