File: pcb/kicad/qwicc_segment_display.kicad_sch (KiCad schematic)
At the start: 2 parts, among them J7 Qwicc Connector

Commit message: rev3-update
Parts:
- J7: value Qwicc Connector -> Qwiic Connector
Other:
- note added: "Qwiic Connector"
- note removed: "Qwicc Connector"
Changed lines of the file:
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@@
   (title_block
     (title "Kwartzlab Environmental Sensor")
-    (date "2023-04-04")
-    (rev "2")
+    (date "2023-04-20")
+    (rev "3")
     (company "Created By: Erin Reed (FireLabs - www.firelabs.ca)")
   )
@@
     (fill (type none))
   )
-  (text "Qwicc Connector" (at 119.38 85.09 0)
+  (text "Qwiic Connector" (at 119.38 85.09 0)
     (effects (font (size 2.27 2.27) (thickness 0.454) bold) (justify left bottom))
   )
@@
     (pin "1")
     (instances
-      (project "KwartzLab-SensorBoard-Rev2"
+      (project "KwartzLab-SensorBoard-Rev3"
         (path "/02789d54-6086-45b9-8196-8325e6f33099/0426278e-287b-42da-b642-f38dcb7eb1f5"
           (reference "#PWR057") (unit 1)
@@
     (pin "1")
     (instances
-      (project "KwartzLab-SensorBoard-Rev2"
+      (project "KwartzLab-SensorBoard-Rev3"
         (path "/02789d54-6086-45b9-8196-8325e6f33099/0426278e-287b-42da-b642-f38dcb7eb1f5"
           (reference "#PWR058") (unit 1)
@@
       (effects (font (size 1.27 1.27)) (justify left))
     )
-    (property "Value" "Qwicc Connector" (at 137.16 92.075 0)
+    (property "Value" "Qwiic Connector" (at 137.16 92.075 0)
       (effects (font (size 1.27 1.27)) (justify left))
     )
@@
     (pin "4")
     (instances
-      (project "KwartzLab-SensorBoard-Rev2"
+      (project "KwartzLab-SensorBoard-Rev3"
         (path "/02789d54-6086-45b9-8196-8325e6f33099/0426278e-287b-42da-b642-f38dcb7eb1f5"
           (reference "J7") (unit 1)
@@
     (pin "2")
     (instances
-      (project "KwartzLab-SensorBoard-Rev2"
+      (project "KwartzLab-SensorBoard-Rev3"
         (path "/02789d54-6086-45b9-8196-8325e6f33099/2426fcd9-5a43-41a7-b855-a8909e878faf"
           (reference "C1") (unit 1)
