File: pcb/kicad/sensor_bme688.kicad_sch (KiCad schematic)
At the start: 3 parts, among them U4 BME688

Commit message: rev3-update
Connections:
- net GND: now also U4.5 (SDO); no longer U4.3 (SDI)
- net SDA: now also U4.3 (SDI); no longer U4.5 (SDO)
Changed lines of the file:
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@@
   (title_block
     (title "Kwartzlab Environmental Sensor")
-    (date "2023-04-04")
-    (rev "2")
+    (date "2023-04-20")
+    (rev "3")
     (company "Created By: Erin Reed (FireLabs - www.firelabs.ca)")
   )
@@
     (stroke (width 0) (type default))
   )
-  (wire (pts (xy 158.75 90.17) (xy 166.37 90.17))
+  (wire (pts (xy 158.75 100.33) (xy 166.37 100.33))
     (stroke (width 0) (type default))
   )
@@
     (stroke (width 0) (type default))
   )
+  (wire (pts (xy 158.75 90.17) (xy 181.61 90.17))
+    (stroke (width 0) (type default))
+  )
   (wire (pts (xy 146.05 115.57) (xy 146.05 118.11))
     (stroke (width 0) (type default))
   )
   (wire (pts (xy 161.29 105.41) (xy 161.29 109.22))
-    (stroke (width 0) (type default))
-  )
-  (wire (pts (xy 158.75 100.33) (xy 181.61 100.33))
     (stroke (width 0) (type default))
   )
@@
     (effects (font (size 2.27 2.27) (thickness 0.454) bold) (justify left bottom))
   )
-  (text "I2C Address Selection" (at 160.02 100.33 0)
+  (text "I2C Address Selection" (at 160.02 88.9 0)
     (effects (font (size 1.27 1.27)) (justify left bottom))
   )
@@
     (effects (font (size 1.27 1.27)) (justify left))
   )
-  (hierarchical_label "SDA" (shape bidirectional) (at 166.37 90.17 0) (fields_autoplaced)
+  (hierarchical_label "SDA" (shape bidirectional) (at 166.37 100.33 0) (fields_autoplaced)
     (effects (font (size 1.27 1.27)) (justify left))
   )
-  (symbol (lib_id "power:GND") (at 181.61 100.33 90) (unit 1)
-    (in_bom yes) (on_board yes) (dnp no) (fields_autoplaced)
-    (property "Reference" "#PWR042" (at 187.96 100.33 0)
-      (effects (font (size 1.27 1.27)) hide)
-    )
-    (property "Value" "GND" (at 185.42 100.965 90)
-      (effects (font (size 1.27 1.27)) (justify right))
-    )
-    (property "Footprint" "" (at 181.61 100.33 0)
-      (effects (font (size 1.27 1.27)) hide)
-    )
-    (property "Datasheet" "" (at 181.61 100.33 0)
-      (effects (font (size 1.27 1.27)) hide)
-    )
-    (pin "1")
-    (instances
-      (project "KwartzLab-SensorBoard-Rev2"
+  (symbol (lib_id "power:GND") (at 181.61 90.17 90) (unit 1)
+    (in_bom yes) (on_board yes) (dnp no) (fields_autoplaced)
+    (property "Reference" "#PWR042" (at 187.96 90.17 0)
+      (effects (font (size 1.27 1.27)) hide)
+    )
+    (property "Value" "GND" (at 185.42 90.805 90)
+      (effects (font (size 1.27 1.27)) (justify right))
+    )
+    (property "Footprint" "" (at 181.61 90.17 0)
+      (effects (font (size 1.27 1.27)) hide)
+    )
+    (property "Datasheet" "" (at 181.61 90.17 0)
+      (effects (font (size 1.27 1.27)) hide)
+    )
+    (pin "1")
+    (instances
+      (project "KwartzLab-SensorBoard-Rev3"
         (path "/02789d54-6086-45b9-8196-8325e6f33099/a3ca797d-6e88-4dc2-831e-93151a2e3212"
           (reference "#PWR042") (unit 1)
@@
     (pin "1")
     (instances
-      (project "KwartzLab-SensorBoard-Rev2"
+      (project "KwartzLab-SensorBoard-Rev3"
         (path "/02789d54-6086-45b9-8196-8325e6f33099/c36effe9-aa4f-4169-b808-b0055ccb3a92"
           (reference "#PWR014") (unit 1)
@@
     (pin "1")
     (instances
-      (project "KwartzLab-SensorBoard-Rev2"
+      (project "KwartzLab-SensorBoard-Rev3"
         (path "/02789d54-6086-45b9-8196-8325e6f33099/a3ca797d-6e88-4dc2-831e-93151a2e3212"
           (reference "#PWR039") (unit 1)
@@
     (pin "1")
     (instances
-      (project "KwartzLab-SensorBoard-Rev2"
+      (project "KwartzLab-SensorBoard-Rev3"
         (path "/02789d54-6086-45b9-8196-8325e6f33099/a3ca797d-6e88-4dc2-831e-93151a2e3212"
           (reference "#PWR040") (unit 1)
@@
     (pin "2")
     (instances
-      (project "KwartzLab-SensorBoard-Rev2"
+      (project "KwartzLab-SensorBoard-Rev3"
         (path "/02789d54-6086-45b9-8196-8325e6f33099/c36effe9-aa4f-4169-b808-b0055ccb3a92"
           (reference "C6") (unit 1)
@@
     (pin "2")
     (instances
-      (project "KwartzLab-SensorBoard-Rev2"
+      (project "KwartzLab-SensorBoard-Rev3"
         (path "/02789d54-6086-45b9-8196-8325e6f33099/c36effe9-aa4f-4169-b808-b0055ccb3a92"
           (reference "C6") (unit 1)
@@
     (pin "1")
     (instances
-      (project "KwartzLab-SensorBoard-Rev2"
+      (project "KwartzLab-SensorBoard-Rev3"
         (path "/02789d54-6086-45b9-8196-8325e6f33099/c36effe9-aa4f-4169-b808-b0055ccb3a92"
           (reference "#PWR014") (unit 1)
@@
     (pin "1")
     (instances
-      (project "KwartzLab-SensorBoard-Rev2"
+      (project "KwartzLab-SensorBoard-Rev3"
         (path "/02789d54-6086-45b9-8196-8325e6f33099/a3ca797d-6e88-4dc2-831e-93151a2e3212"
           (reference "#PWR036") (unit 1)
@@
     (pin "1")
     (instances
-      (project "KwartzLab-SensorBoard-Rev2"
+      (project "KwartzLab-SensorBoard-Rev3"
         (path "/02789d54-6086-45b9-8196-8325e6f33099/a3ca797d-6e88-4dc2-831e-93151a2e3212"
           (reference "#PWR041") (unit 1)
@@
     (pin "1")
     (instances
-      (project "KwartzLab-SensorBoard-Rev2"
+      (project "KwartzLab-SensorBoard-Rev3"
         (path "/02789d54-6086-45b9-8196-8325e6f33099/a3ca797d-6e88-4dc2-831e-93151a2e3212"
           (reference "#PWR038") (unit 1)
@@
     (pin "8")
     (instances
-      (project "KwartzLab-SensorBoard-Rev2"
+      (project "KwartzLab-SensorBoard-Rev3"
         (path "/02789d54-6086-45b9-8196-8325e6f33099/a3ca797d-6e88-4dc2-831e-93151a2e3212"
           (reference "U4") (unit 1)
