File: pcb/kicad/KwartzLab-SensorBoard-Rev3-Panel.kicad_pcb (KiCad board)
At the start: 2 copper layers, 185.9 x 120 mm, 198 parts, among them J1 Serial Interface, J2 USB_C_Receptacle_USB2.0, J3 PM2.5 Sensor, J4 Zio Loudness Sensor, J5 Screw_Terminal_01x03, J6 Screw_Terminal_01x03, J7 Qwiic Connector, J8 Conn_02x02_Odd_Even, J9 Conn_02x02_Odd_Even, K1 5v Relay, K2 5v Relay, Q1 MMBT3904, Q2 MMBT3904, SW1 SW_Push, SW2 SW_Push, U1 ESP32-C3-MINI-1, U2 AMS1117-3.3, U3 SHTC3, U4 BME688

Commit message: updated a few parts
Parts:
- removed the D6 at (142.6, 83.8)
- removed the D6 at (52.7, 83.8)
- removed the D7 at (160.8, 83.8)
- removed the D7 at (70.9, 83.8)
- removed the REF** at (52.2, 22.5) (x2)
- removed the REF** at (52.2, 131.5) (x2)
- removed the REF** at (227.2, 22.5) (x2)
- added ?: , , F.Cu at (142.6, 81.5)
- added ?: , , F.Cu at (52.7, 81.5)
- added D6: LL4148, LL4148:DIO_LL4148, F.Cu at (52.7, 83.4)
- added D6: LL4148, LL4148:DIO_LL4148, F.Cu at (142.6, 83.4)
- added D7: LL4148, LL4148:DIO_LL4148, F.Cu at (160.9, 83.4)
- added D7: LL4148, LL4148:DIO_LL4148, F.Cu at (70.9, 83.4)
- added REF**: Fiducial, Fiducial, F.Cu at (52.2, 22.5)
- added REF**: Fiducial, Fiducial, B.Cu at (227.2, 22.5)
- added REF**: Fiducial, Fiducial, B.Cu at (52.2, 131.5)
- added REF**: Fiducial, Fiducial, B.Cu at (52.2, 22.5)
- added REF**: Fiducial, Fiducial, F.Cu at (227.2, 22.5)
- added REF**: Fiducial, Fiducial, F.Cu at (52.2, 131.5)
Routing:
- net Board_0-GND: track 101.9 -> 97.7 mm
- net Board_1-GND: track 101.9 -> 97.7 mm
- net Board_1-+5V: track 217.3 -> 216.3 mm
- net Board_0-+5V: track 217.3 -> 216.3 mm
- net Board_1-/Output Relays/RELAY2_EN: track 28.2 -> 27.6 mm
- net Board_0-/Output Relays/RELAY2_EN: track 28.2 -> 27.6 mm
