File: pcb/kicad/KwartzLab-SensorBoard-Rev3.kicad_pcb (KiCad board)
At the start: 2 copper layers, 90 x 100 mm, 94 parts, among them J1 Serial Interface, J2 USB_C_Receptacle_USB2.0, J3 PM2.5 Sensor, J4 Zio Loudness Sensor, J5 Screw_Terminal_01x03, J6 Screw_Terminal_01x03, J7 Qwiic Connector, J8 Conn_02x02_Odd_Even, J9 Conn_02x02_Odd_Even, K1 5v Relay, K2 5v Relay, Q1 MMBT3904, Q2 MMBT3904, SW1 SW_Push, SW2 SW_Push, U1 ESP32-C3-MINI-1, U2 AMS1117-3.3, U3 SHTC3, U4 BME688

Commit message: updated a few parts
Parts:
- added ?: , , F.Cu at (93.0, 113.1)
- D6, D7: value 1N4148W -> LL4148; footprint Diode_SMD:D_SOD-123 -> LL4148:DIO_LL4148
- moved D6 0.42 mm to (93.0, 115.1)
- moved D7 0.37 mm to (111.3, 115.1)
Routing:
- net GND: track 101.9 -> 97.7 mm
- net +5V: track 217.3 -> 216.3 mm
- net /Output Relays/RELAY2_EN: track 28.2 -> 27.6 mm
